File: elec/RaceCard/power.kicad_sch (KiCad schematic)
At the start: 0 parts

Commit message: ajout de reverse polarity et efuse
Parts:
- added C1, C2: 1uF, Capacitor_SMD:C_0603_1608Metric, symbol Device:C_Small
- added D1: D_Schottky_Small, symbol Device:D_Schottky_Small
- added F1: 0ZCJ0025FF2E, C3I_A25:0ZCJ_BEL, symbol C3I_A25:0ZCJ0025FF2E
- added Q1: DMP3125L-7, C3I_A25:SOT91P240X110-3N, symbol Transistor_FET:Q_PMOS_GSD
- added U1: TLV74033PDQNR, C3I_A25:SUP_TPS3831L30DQNR, symbol C3I_A25:TLV74033PDQNR
Connections:
- new net: C2.1, D1.2 (A), U1.1 (OUT)
- new net: F1.2, Q1.3 (D)
- new net: C1.1, D1.1 (K), Q1.2 (S), U1.3 (EN), U1.4 (IN)
- new net GND: C1.2, C2.2, Q1.1 (G), U1.2 (GND)
Other:
- note added: "Vérifier la nécessité"

Commit message: V1 du chargeur fini
Valider par qqn d'autre que Hugo
Parts:
- added C3: 1uF, Capacitor_SMD:C_0603_1608Metric, symbol Device:C_Small
- added C4: 4.7uF, Capacitor_SMD:C_0603_1608Metric, symbol Device:C_Small
- added J1: 530480210, 530480210:MOLEX_530480210, symbol C3I_A25:530480210
- added R1: 10k, Resistor_SMD:R_0603_1608Metric, symbol Device:R_Small_US
- added U2: MCP73812T-420I_OT, MCP73812T-420I_OT:SOT95P280X145-5N, symbol C3I_A25:MCP73812T-420I_OT
- added U3: AS11AH, AS11AH:AS11AH, symbol C3I_A25:AS11AH
Connections:
- net GND: now also C3.2, C4.2, J1.1 (-), R1.2, U2.2 (VSS)
- net at F1.1: now also C4.1, U2.3 (VBAT), U3.2
- new net: R1.1, U2.5 (PROG)
- new net: J1.2 (+), U3.1
- new net: C3.1, U2.1 (CE), U2.4 (VDD)
Other:
- note added: "Pour I_charge de 100 mA"
- moved on the sheet: C1, C2, D1, F1, Q1, U1
