File: elec/RaceCard/power.kicad_sch (KiCad schematic)
At the start: 26 parts, among them J2 UJC-H-G-SMT-2-P6-TR, J3 530480210, Q1 DMP3125L-7, U3 MCP73812T-420I_OT, U4 TLV74033PDQNR, U5 AS11AH

Commit message: Manque juste RF
Connections:
- net VIN: now reaches C21.1, D2.1 (K), Q1.2 (S), TP15.1, U4.3 (EN), U4.4 (IN)
- net VBAT: now reaches C17.1, F1.1, TP14.1, U3.3 (VBAT), U5.2
- net VBUS: now reaches C18.1, C19.1, C20.1, CR1.1, J2.A9 (VBUS), J2.B9 (VBUS__1), R12.1, TP13.1, U3.1 (CE), U3.4 (VDD)

Commit message: Cleanup
Other:
- moved on the sheet: C17, C18, C19, C20, C21, C22, CR1, D1, D2, D3, F1, J2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
