File: elec/RaceCard/stm32.kicad_sch (KiCad schematic)
At the start: 0 parts

Commit message: Ajout du schema à gab
Parts:
- added C1: 4.7uF, symbol Device:C
- added C2, C3, C4, C5: 100nF, symbol Device:C
- added C6: 1uF, symbol Device:C
- added C7: 10nF, symbol Device:C
- added J1: Conn_ST_STDC14, C3I:CONN_3020-14-0300-00_CNC, symbol Connector:Conn_ST_STDC14
- added R1: R0, symbol Device:R_US
- added U1: STM32U031C6Tx, Package_QFP:LQFP-48_7x7mm_P0.5mm, symbol MCU_ST_STM32U0:STM32U031C6Tx
Connections:
- new net AGND: C6.2, C7.2, U1.8 (VSSA)
- new net GND: C1.2, C2.2, C3.2, C4.2, C5.2, J1.11 (GNDDetect), J1.5 (GND), J1.7 (GND), U1.23 (VSS), U1.35 (VSS), U1.47 (VSS)
- new net NRST: J1.12 (~{RST}), U1.7 (PF2)
- new net SWCLK: J1.6 (JCLK/SWCLK), U1.37 (PA14)
- new net SWDIO: J1.4 (JTMS/SWDIO), U1.34 (PA13)
- new net VDD: C1.1, C2.1, C3.1, C4.1, C5.1, J1.3 (VCC), R1.1, U1.24 (VDD), U1.36 (VDD), U1.48 (VDD)
- new net VDDA: C6.1, C7.1, R1.2, U1.9 (VDDA)
Other:
- note added: "JTAG CONNECTOR"
- note added: "MCU DECAPS"
- note added: "STM32U031 MCU INITIAL CONNECTIONS"
