File: elec/RaceCard/RaceCard.kicad_pcb (KiCad board)
At the start: 4 copper layers, 85.6 x 54 mm, 79 parts, among them J1 Conn_ST_STDC14, J2 UJC-H-G-SMT-2-P6-TR, J3 530480210, Q1 DMP3125L-7, U1 STM32U031C6Tx, U2 IQS7222A001QFR, U3 MCP73812T-420I_OT, U4 TLV74033PDQNR, U5 AS11AH, U6 MICRF112YMM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

Commit message: Tout le power est routed
Parts:
- moved TP12 175.5 mm to (131.7, 124.7)
- moved TP14 170.3 mm to (142.3, 124.7)
- moved TP13 168.8 mm to (137.0, 124.7)
- moved TP15 163.6 mm to (147.6, 124.7)
- moved R13 143.8 mm to (123.0, 103.8), turned to 90 degrees
- moved U3 139.5 mm to (128.4, 104.0)
- moved R15 136.2 mm to (117.0, 107.3), turned to 180 degrees
- moved R17 133.5 mm to (117.0, 105.8)
- moved CR1 127.5 mm to (128.5, 99.7)
- moved C15 127.3 mm to (123.8, 106.3), turned to 180 degrees
- moved F1 125.8 mm to (120.9, 111.0), turned to 135 degrees
- moved Q1 125.5 mm to (127.1, 111.7), turned to 180 degrees
- moved C17 123.7 mm to (122.3, 100.0), turned to 90 degrees
- moved C16 122.5 mm to (128.5, 107.5), turned to -90 degrees
- moved U4 122.1 mm to (135.0, 105.0), turned to -90 degrees
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Connections:
- C6 pad 1: Net-(C6-Pad1) -> VDDA
- C7 pad 1: Net-(C6-Pad1) -> VDDA
- R1 pad 2: unconnected-(R1-Pad2) -> VDDA
- U1 pad 9: unconnected-(U1-VDDA-Pad9) -> VDDA
- U5 pad P$1: GND -> (no net)
- U5 pad P$3: GND -> (no net)
Routing:
- net /Power/VDD: track 0.00 -> 79.3 mm, vias 0 -> 14
- net Net-(J2-VBUS): track 0.00 -> 55.4 mm, vias 0 -> 1
- net SWDIO: track 0.00 -> 53.9 mm, vias 0 -> 1
- net SWCLK: track 0.00 -> 48.6 mm, vias 0 -> 1
- net GND: track 0.00 -> 42.2 mm, vias 0 -> 28
- net Net-(U3-VBAT): track 0.00 -> 40.3 mm
- net NRST: track 0.00 -> 37.4 mm, vias 0 -> 1
- net Net-(D2-K): track 0.00 -> 31.0 mm, vias 0 -> 2
- net VDDA: track 0.00 -> 8.89 mm, vias 0 -> 2
- net Net-(Q1-D): track 0.00 -> 7.87 mm, vias 0 -> 2
- net Net-(J3-+): track 0.00 -> 7.18 mm
- net Net-(D1-PadC): track 0.00 -> 4.26 mm
- net Net-(J2-CC2): track 0.00 -> 2.34 mm, vias 0 -> 1
- net Net-(J2-CC1): track 0.00 -> 2.33 mm, vias 0 -> 1
- net Net-(U3-PROG): track 0.00 -> 2.03 mm
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- added copper zone on In2.Cu, net /Power/VDD
- added copper zone on In1.Cu, net GND
- added copper zone on In2.Cu, net VDDA
