File: elec/RaceCard/sensors.kicad_sch (KiCad schematic)
At the start: 21 parts, among them U2 IQS7222A001QFR

Commit message: Power net update et cleanup sch
Parts:
- renumbered C8 to C10, C9 to C11, C10 to C12, C11 to C13, C12 to C14, C13 to C15, C14 to C16, R2 to R1, R11 to R10, R12 to R11, R3 to R2, R4 to R3, R5 to R4, R6 to R5, R7 to R6, R8 to R7, R9 to R8, R10 to R9, TP10 to TP11, TP11 to TP12
Connections:
- net VDD renamed +3V3
Other:
- note removed: "3.3V"

Commit message: Manque juste RF
Parts:
- added U10: 4ch_Slider, C3I_A25:4chSlider, symbol C3I_A25:4chSlider
- added U7: BTN1, C3I_A25:BigTouch, symbol C3I_A25:SmallTouch
- added U8: BTN2, C3I_A25:SmallTouch, symbol C3I_A25:SmallTouch
- added U9: BTN3, C3I_A25:SmallTouch, symbol C3I_A25:SmallTouch
Connections:
- net CX0: now also U10.4 (ch4)
- net CX1: now also U10.3 (ch3)
- net CX2: now also U10.2 (ch2)
- net CX3: now also U10.1 (ch1)
- net CX5: now also U7.1 (T)
- net CX6: now also U8.1 (T)
- net CX7: now also U9.1 (T)
Other:
- note added: "I2C address est 0x44 puisque le part number est IQS7222A001CSR (où 001 veut dire 0x44)"
- note added: "The CSP package is sensitive to infrared light. When the silicon IC is subject to the photo-electric effect, an increase in leakage current is experienced. Due to the low power consumption of the IC this causes a change in signal and is common in the semiconductor industry with CSP devices. If the IC could be exposed to IR in the product, then a dark glob-top epoxy material should cover the compl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"

Commit message: Cleanup
Other:
- moved on the sheet: C10, C11, C12, C13, C14, C15, C16, R1, R10, R11, R2, R3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
